Commit message: adding urdf files for erl_drone as well as parameters and xacro generation scripts

File: models/erl_drone/erl_drone.urdf.xacro (robot description, xacro)
@@ -1,12 +1,8 @@
 <?xml version="1.0" ?>
 <!-- =================================================================================== -->
-<!-- |    This document was autogenerated by xacro from erl_base.xacro                 | -->
+<!-- |    This document was autogenerated by xacro from urdf/erl_base_template.xacro   | -->
 <!-- |    EDITING THIS FILE BY HAND IS NOT RECOMMENDED                                 | -->
 <!-- =================================================================================== -->
-<!-- =================================================================================== -->
-<!-- |    This document was autogenerated by xacro from erl_base.xacro                 | -->
-<!-- |    EDITING THIS FILE BY HAND IS NOT RECOMMENDED                                 | -->
-<!-- =================================================================================== -->
-<robot name="iris" xmlns:xacro="http://ros.org/wiki/xacro">
+<robot name="erl_drone" xmlns:xacro="http://ros.org/wiki/xacro">
   <!-- Properties that can be assigned at build time as arguments.
   Is there a reason not to make all properties arguments?
@@ -28,5 +24,5 @@
   <!-- Macro to add a depth camera on the VI-sensor. -->
   <!-- VI-Sensor Macro -->
-  <!-- Instantiate iris "mechanics" -->
+  <!-- Instantiate erl_drone "mechanics" -->
   <!-- Properties -->
   <!-- [kg] -->
@@ -45,6 +41,22 @@
   <!-- [s] -->
   <!-- [rad/s] -->
-  <!-- Property Blocks -->
-  <!-- inertia of a single rotor, assuming it is a cuboid. Height=3mm, width=15mm -->
+  <!-- Property Blocks
+  <xacro:property name="body_inertia">
+    <inertia
+    ixx="${1/12 * mass * (body_height * body_height + body_width * body_width)}"
+    iyy="${1/12 * mass * (body_height * body_height + body_width * body_width)}"
+    izz="${1/12 * mass * (body_width * body_width + body_width * body_width)}"
+    ixy="0.0" ixz="0.0" iyz="0.0" />  [kg.m^2] [kg.m^2] [kg.m^2] [kg.m^2] [kg.m^2] [kg.m^2]
+  </xacro:property>
+  -->
+  <!-- inertia of a single rotor, assuming it is a cuboid. Height=3mm, width=15mm
+  <xacro:property name="rotor_inertia">
+    <inertia
+    ixx="${1/12 * mass_rotor * (0.015 * 0.015 + 0.003 * 0.003) * rotor_velocity_slowdown_sim}"
+    iyy="${1/12 * mass_rotor * (4 * radius_rotor * radius_rotor + 0.003 * 0.003) * rotor_velocity_slowdown_sim}"
+    izz="${1/12 * mass_rotor * (4 * radius_rotor * radius_rotor + 0.015 * 0.015) * rotor_velocity_slowdown_sim}"
+    ixy="0.0" ixz="0.0"  iyz="0.0" /> [kg.m^2] [kg.m^2] [kg.m^2] [kg.m^2] [kg.m^2] [kg.m^2]
+  </xacro:property>
+  -->
   <!-- Included URDF Files -->
   <!-- Main multirotor link -->
@@ -62,10 +74,10 @@
       <!-- [kg] -->
       <origin xyz="0 0 0"/>
-      <inertia ixx="0.029124999999999998" ixy="0.0" ixz="0.0" iyy="0.029124999999999998" iyz="0.0" izz="0.055224999999999996"/>
+      <inertia ixx="0.011994" ixy="0.0" ixz="0.0" iyy="0.011226" iyz="0.0" izz="0.019944"/>
     </inertial>
     <visual>
       <origin rpy="0 0 0" xyz="0 0 0"/>
       <geometry>
-        <mesh filename="model://iris/meshes/iris.stl" scale="1 1 1"/>
+        <mesh filename="model://erl_drone/meshes/erl_drone.stl" scale="1 1 1"/>
         <!-- <box size="${body_width} ${body_width} ${body_height}"/> -->
         <!-- [m] [m] [m] -->
@@ -75,5 +87,5 @@
       <origin rpy="0 0 0" xyz="0 0 0"/>
       <geometry>
-        <box size="0.47 0.47 0.11"/>
+        <box size="0.5 0.5 0.18"/>
         <!-- [m] [m] [m] -->
       </geometry>
@@ -83,5 +95,5 @@
   <gazebo>
     <plugin filename="libgazebo_multirotor_base_plugin.so" name="rosbag">
-      <robotNamespace/>
+      <robotNamespace></robotNamespace>
       <linkName>base_link</linkName>
       <rotorVelocitySlowdownSim>10</rotorVelocitySlowdownSim>
@@ -106,5 +118,5 @@
   <!-- Instantiate rotors -->
   <joint name="rotor_0_joint" type="continuous">
-    <origin rpy="0 0 0" xyz="0.13 -0.22 0.023"/>
+    <origin rpy="0 0 0" xyz="0.175 -0.175 0.075"/>
     <axis xyz="0 0 1"/>
     <!-- TODO(ff): not currently set because it's not yet supported -->
@@ -120,5 +132,5 @@
       <mass value="0.005"/>
       <!-- [kg] -->
-      <inertia ixx="9.75e-07" ixy="0.0" ixz="0.0" iyy="0.0002731041666666666" iyz="0.0" izz="0.0002740041666666667"/>
+      <inertia ixx="9.75e-07" ixy="0.0" ixz="0.0" iyy="0.000273104" iyz="0.0" izz="0.000274004"/>
     </inertial>
     <visual>
@@ -127,5 +139,5 @@
         <!-- [m] -->
         <!-- <mesh filename="package://rotors_description/meshes/propeller_${direction}.dae" -->
-        <mesh filename="model://iris/meshes/iris_prop_ccw.dae" scale="1 1 1"/>
+        <mesh filename="model://erl_drone/meshes/iris_prop_ccw.dae" scale="1 1 1"/>
         <!-- <box size="${2*radius_rotor} 0.01 0.005"/> -->
       </geometry>
@@ -140,5 +152,5 @@
   <gazebo>
     <plugin filename="libgazebo_motor_model.so" name="front_right_motor_model">
-      <robotNamespace/>
+      <robotNamespace></robotNamespace>
       <jointName>rotor_0_joint</jointName>
       <linkName>rotor_0</linkName>
@@ -146,7 +158,7 @@
       <timeConstantUp>0.0125</timeConstantUp>
       <timeConstantDown>0.025</timeConstantDown>
-      <maxRotVelocity>1100</maxRotVelocity>
-      <motorConstant>8.54858e-06</motorConstant>
-      <momentConstant>0.06</momentConstant>
+      <maxRotVelocity>1000</maxRotVelocity>
+      <motorConstant>5.46e-06</motorConstant>
+      <momentConstant>0.0158</momentConstant>
       <commandSubTopic>/gazebo/command/motor_speed</commandSubTopic>
       <motorNumber>0</motorNumber>
@@ -172,5 +184,5 @@
   </gazebo>
   <joint name="rotor_1_joint" type="continuous">
-    <origin rpy="0 0 0" xyz="-0.13 0.2 0.023"/>
+    <origin rpy="0 0 0" xyz="-0.175 0.175 0.075"/>
     <axis xyz="0 0 1"/>
     <!-- TODO(ff): not currently set because it's not yet supported -->
@@ -186,5 +198,5 @@
       <mass value="0.005"/>
       <!-- [kg] -->
-      <inertia ixx="9.75e-07" ixy="0.0" ixz="0.0" iyy="0.0002731041666666666" iyz="0.0" izz="0.0002740041666666667"/>
+      <inertia ixx="9.75e-07" ixy="0.0" ixz="0.0" iyy="0.000273104" iyz="0.0" izz="0.000274004"/>
     </inertial>
     <visual>
@@ -193,5 +205,5 @@
         <!-- [m] -->
         <!-- <mesh filename="package://rotors_description/meshes/propeller_${direction}.dae" -->
-        <mesh filename="model://iris/meshes/iris_prop_ccw.dae" scale="1 1 1"/>
+        <mesh filename="model://erl_drone/meshes/iris_prop_ccw.dae" scale="1 1 1"/>
         <!-- <box size="${2*radius_rotor} 0.01 0.005"/> -->
       </geometry>
@@ -206,5 +218,5 @@
   <gazebo>
     <plugin filename="libgazebo_motor_model.so" name="back_left_motor_model">
-      <robotNamespace/>
+      <robotNamespace></robotNamespace>
       <jointName>rotor_1_joint</jointName>
       <linkName>rotor_1</linkName>
@@ -212,7 +224,7 @@
       <timeConstantUp>0.0125</timeConstantUp>
       <timeConstantDown>0.025</timeConstantDown>
-      <maxRotVelocity>1100</maxRotVelocity>
-      <motorConstant>8.54858e-06</motorConstant>
-      <momentConstant>0.06</momentConstant>
+      <maxRotVelocity>1000</maxRotVelocity>
+      <motorConstant>5.46e-06</motorConstant>
+      <momentConstant>0.0158</momentConstant>
       <commandSubTopic>/gazebo/command/motor_speed</commandSubTopic>
       <motorNumber>1</motorNumber>
@@ -238,5 +250,5 @@
   </gazebo>
   <joint name="rotor_2_joint" type="continuous">
-    <origin rpy="0 0 0" xyz="0.13 0.22 0.023"/>
+    <origin rpy="0 0 0" xyz="0.175 0.175 0.075"/>
     <axis xyz="0 0 1"/>
     <!-- TODO(ff): not currently set because it's not yet supported -->
@@ -252,5 +264,5 @@
       <mass value="0.005"/>
       <!-- [kg] -->
-      <inertia ixx="9.75e-07" ixy="0.0" ixz="0.0" iyy="0.0002731041666666666" iyz="0.0" izz="0.0002740041666666667"/>
+      <inertia ixx="9.75e-07" ixy="0.0" ixz="0.0" iyy="0.000273104" iyz="0.0" izz="0.000274004"/>
     </inertial>
     <visual>
@@ -259,5 +271,5 @@
         <!-- [m] -->
         <!-- <mesh filename="package://rotors_description/meshes/propeller_${direction}.dae" -->
-        <mesh filename="model://iris/meshes/iris_prop_cw.dae" scale="1 1 1"/>
+        <mesh filename="model://erl_drone/meshes/iris_prop_cw.dae" scale="1 1 1"/>
         <!-- <box size="${2*radius_rotor} 0.01 0.005"/> -->
       </geometry>
@@ -272,5 +284,5 @@
   <gazebo>
     <plugin filename="libgazebo_motor_model.so" name="front_left_motor_model">
-      <robotNamespace/>
+      <robotNamespace></robotNamespace>
       <jointName>rotor_2_joint</jointName>
       <linkName>rotor_2</linkName>
@@ -278,7 +290,7 @@
       <timeConstantUp>0.0125</timeConstantUp>
       <timeConstantDown>0.025</timeConstantDown>
-      <maxRotVelocity>1100</maxRotVelocity>
-      <motorConstant>8.54858e-06</motorConstant>
-      <momentConstant>0.06</momentConstant>
+      <maxRotVelocity>1000</maxRotVelocity>
+      <motorConstant>5.46e-06</motorConstant>
+      <momentConstant>0.0158</momentConstant>
       <commandSubTopic>/gazebo/command/motor_speed</commandSubTopic>
       <motorNumber>2</motorNumber>
@@ -304,5 +316,5 @@
   </gazebo>
   <joint name="rotor_3_joint" type="continuous">
-    <origin rpy="0 0 0" xyz="-0.13 -0.2 0.023"/>
+    <origin rpy="0 0 0" xyz="-0.175 -0.175 0.075"/>
     <axis xyz="0 0 1"/>
     <!-- TODO(ff): not currently set because it's not yet supported -->
@@ -318,5 +330,5 @@
       <mass value="0.005"/>
       <!-- [kg] -->
-      <inertia ixx="9.75e-07" ixy="0.0" ixz="0.0" iyy="0.0002731041666666666" iyz="0.0" izz="0.0002740041666666667"/>
+      <inertia ixx="9.75e-07" ixy="0.0" ixz="0.0" iyy="0.000273104" iyz="0.0" izz="0.000274004"/>
     </inertial>
     <visual>
@@ -325,5 +337,5 @@
         <!-- [m] -->
         <!-- <mesh filename="package://rotors_description/meshes/propeller_${direction}.dae" -->
-        <mesh filename="model://iris/meshes/iris_prop_cw.dae" scale="1 1 1"/>
+        <mesh filename="model://erl_drone/meshes/iris_prop_cw.dae" scale="1 1 1"/>
         <!-- <box size="${2*radius_rotor} 0.01 0.005"/> -->
       </geometry>
@@ -338,5 +350,5 @@
   <gazebo>
     <plugin filename="libgazebo_motor_model.so" name="back_right_motor_model">
-      <robotNamespace/>
+      <robotNamespace></robotNamespace>
       <jointName>rotor_3_joint</jointName>
       <linkName>rotor_3</linkName>
@@ -344,7 +356,7 @@
       <timeConstantUp>0.0125</timeConstantUp>
       <timeConstantDown>0.025</timeConstantDown>
-      <maxRotVelocity>1100</maxRotVelocity>
-      <motorConstant>8.54858e-06</motorConstant>
-      <momentConstant>0.06</momentConstant>
+      <maxRotVelocity>1000</maxRotVelocity>
+      <motorConstant>5.46e-06</motorConstant>
+      <momentConstant>0.0158</momentConstant>
       <commandSubTopic>/gazebo/command/motor_speed</commandSubTopic>
       <motorNumber>3</motorNumber>
@@ -372,5 +384,5 @@
   <gazebo>
     <plugin filename="libgazebo_gps_plugin.so" name="gps_plugin">
-      <robotNamespace/>
+      <robotNamespace></robotNamespace>
       <gpsNoise>true</gpsNoise>
     </plugin>
@@ -379,5 +391,5 @@
   <gazebo>
     <plugin filename="libgazebo_magnetometer_plugin.so" name="magnetometer_plugin">
-      <robotNamespace/>
+      <robotNamespace></robotNamespace>
       <pubRate>20</pubRate>
       <noiseDensity>0.0004</noiseDensity>
@@ -390,5 +402,5 @@
   <gazebo>
     <plugin filename="libgazebo_barometer_plugin.so" name="barometer_plugin">
-      <robotNamespace/>
+      <robotNamespace></robotNamespace>
       <pubRate>10</pubRate>
       <baroTopic>/baro</baroTopic>
@@ -398,5 +410,5 @@
   <gazebo>
     <plugin filename="libgazebo_mavlink_interface.so" name="mavlink_interface">
-      <robotNamespace/>
+      <robotNamespace></robotNamespace>
       <imuSubTopic>/imu</imuSubTopic>
       <gpsSubTopic>/gps</gpsSubTopic>
@@ -542,5 +554,5 @@
       <!-- A good description of the IMU parameters can be found in the kalibr documentation:
            https://github.com/ethz-asl/kalibr/wiki/IMU-Noise-Model-and-Intrinsics -->
-      <robotNamespace/>
+      <robotNamespace></robotNamespace>
       <!-- (string, required): ros namespace in which the messages are published -->
       <linkName>/imu_link</linkName>

File: models/rotors_description/urdf/erl_drone.xacro (robot description, xacro)
@@ -61,5 +61,5 @@
   -->
   <!-- Included URDF Files -->
-  <xacro:include filename="$(arg rotors_description_dir)/urdf/multirotor_base.xacro" />
+  <xacro:include filename="$(arg rotors_description_dir)/urdf/erl_multirotor_base.xacro" />
   <!-- Instantiate multirotor_base_macro once -->
   <xacro:multirotor_base_macro
